File: tmtua.kicad_sch (KiCad schematic)
At the start: 6 parts, among them CN1 HF1004E, CN2 HF1004E, J1 B-2100S08P-A110, J2 B-2100S08P-A110, J3 PZ200V-11-03P, J4 PZ200V-11-03P

Commit message: correct schematic
Parts:
- J1, J2: symbol Connector:Conn_01x08_Socket -> Connector:Conn_01x08_Pin
Changed lines of the file:
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@@
 	)
 	(symbol
-		(lib_id "Connector:Conn_01x08_Socket")
+		(lib_id "Connector:Conn_01x08_Pin")
 		(at 74.93 59.69 0)
+		(mirror y)
 		(unit 1)
 		(exclude_from_sim no)
@@
 		(dnp no)
 		(property "Reference" "J1"
-			(at 73.406 50.292 0)
+			(at 76.454 50.292 0)
 			(effects
 				(font
@@
 		)
 		(property "Value" "B-2100S08P-A110"
-			(at 76.2 61.468 90)
+			(at 73.66 61.468 90)
 			(effects
 				(font
@@
 	)
 	(symbol
-		(lib_id "Connector:Conn_01x08_Socket")
+		(lib_id "Connector:Conn_01x08_Pin")
 		(at 83.82 59.69 0)
-		(mirror y)
 		(unit 1)
 		(exclude_from_sim no)
@@
 		)
 		(property "Value" "B-2100S08P-A110"
-			(at 82.296 61.468 90)
-			(effects
-				(font
+			(at 85.344 61.468 90)
+			(effects
+				(font
